File: ext-charger.kicad_pcb (KiCad board)
At the start: 2 copper layers, 530 x 170 mm, 61 parts, among them J1 1714971, J10 B2B-PH-K-S, J11 B2B-PH-K-S, J12 B2B-PH-K-S, J13 B2B-PH-K-S, J14 B2B-PH-K-S, J15 B2B-PH-K-S, J16 B2B-PH-K-S, J17 B2B-PH-K-S, J18 B2B-PH-K-S, J19 B2B-PH-K-S, J2 B2B-PH-K-S, J20 B2B-PH-K-S, J21 B2B-PH-K-S, J3 B2B-PH-K-S, J4 B2B-PH-K-S, J5 B2B-PH-K-S, J6 B2B-PH-K-S, J7 B2B-PH-K-S, J8 B2B-PH-K-S, J9 B2B-PH-K-S, U1 TP4056, U10 TP4056, U11 TP4056, U12 TP4056, U13 TP4056, U14 TP4056, U15 TP4056, U16 TP4056, U17 TP4056, U18 TP4056, U19 TP4056, U2 TP4056, U20 TP4056, U3 TP4056, U4 TP4056, U5 TP4056, U6 TP4056, U7 TP4056, U8 TP4056, U9 TP4056

Commit message: finished component placement
Parts:
- moved U19 325.2 mm to (482.3, 210.0), turned to 90 degrees
- moved U20 304.0 mm to (532.3, 210.0), turned to 90 degrees
- moved H11 294.7 mm to (68.9, 195.9)
- moved J10 292.0 mm to (552.5, 125.7)
- moved J9 290.2 mm to (502.5, 125.7)
- moved J20 284.6 mm to (552.5, 203.7)
- moved U18 282.6 mm to (432.3, 210.0), turned to 90 degrees
- moved U10 280.9 mm to (532.3, 132.0), turned to 90 degrees
- moved H20 270.8 mm to (518.9, 195.9)
- moved J19 251.3 mm to (502.5, 203.7)
- moved J12 251.2 mm to (152.5, 203.7)
- moved H1 248.2 mm to (68.9, 117.9)
- moved U9 242.8 mm to (482.3, 132.0), turned to 90 degrees
- moved U1 240.8 mm to (82.3, 132.0), turned to 90 degrees
- moved H13 234.7 mm to (168.9, 195.9)
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- renumbered J2 to J1, J11 to J10, J12 to J11, J13 to J12, J14 to J13, J15 to J14, J16 to J15, J17 to J16, J18 to J17, J19 to J18, J20 to J19, J3 to J2, J21 to J20, J4 to J3, J5 to J4, J6 to J5, J7 to J6, J8 to J7, J9 to J8, J10 to J9
Other:
- outline, holes or cut-outs redrawn

Commit message: finished routing
Routing:
- net /5V: track 0.00 -> 1333.9 mm
- net /GND: track 0.00 -> 1293.2 mm
- net Net-(J5-Pad2): track 0.00 -> 21.9 mm
- net Net-(J20-Pad2): track 0.00 -> 21.2 mm
- net Net-(J2-Pad2): track 0.00 -> 20.5 mm
- net Net-(J4-Pad2): track 0.00 -> 20.4 mm
- net Net-(J17-Pad2): track 0.00 -> 20.0 mm
- net Net-(J19-Pad2): track 0.00 -> 19.9 mm
- net Net-(J18-Pad2): track 0.00 -> 19.6 mm
- net Net-(J12-Pad2): track 0.00 -> 19.5 mm
- net Net-(J13-Pad2): track 0.00 -> 19.5 mm
- net Net-(J15-Pad2): track 0.00 -> 19.5 mm
- net Net-(J11-Pad2): track 0.00 -> 19.3 mm
- net Net-(J8-Pad2): track 0.00 -> 19.2 mm
- net Net-(J14-Pad2): track 0.00 -> 19.2 mm
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
Commit message: added filled zones
Parts:
- renumbered J9 to J10, J10 to J11, J11 to J12, J12 to J13, J13 to J14, J14 to J15, J15 to J16, J16 to J17, J17 to J18, J18 to J19, J1 to J2, J19 to J20, J20 to J21, J2 to J3, J3 to J4, J4 to J5, J5 to J6, J6 to J7, J7 to J8, J8 to J9
Connections:
- J10 pad 2: Net-(J10-Pad2) -> /GND
- J11 pad 2: Net-(J11-Pad2) -> /GND
- J12 pad 2: Net-(J12-Pad2) -> /GND
- J13 pad 2: Net-(J13-Pad2) -> /GND
- J14 pad 2: Net-(J14-Pad2) -> /GND
- J15 pad 2: Net-(J15-Pad2) -> /GND
- J16 pad 2: Net-(J16-Pad2) -> /GND
- J17 pad 2: Net-(J17-Pad2) -> /GND
- J18 pad 2: Net-(J18-Pad2) -> /GND
- J19 pad 2: Net-(J19-Pad2) -> /GND
- J2 pad 2: Net-(J2-Pad2) -> /GND
- J20 pad 2: Net-(J20-Pad2) -> /GND
- J21 pad 2: Net-(J21-Pad2) -> /GND
- J3 pad 2: Net-(J3-Pad2) -> /GND
- J4 pad 2: Net-(J4-Pad2) -> /GND
- J5 pad 2: Net-(J5-Pad2) -> /GND
- J6 pad 2: Net-(J6-Pad2) -> /GND
- J7 pad 2: Net-(J7-Pad2) -> /GND
- J8 pad 2: Net-(J8-Pad2) -> /GND
- J9 pad 2: Net-(J9-Pad2) -> /GND
- U1 pad 4: Net-(J2-Pad2) -> /GND
- U10 pad 4: Net-(J11-Pad2) -> /GND
- U11 pad 4: Net-(J12-Pad2) -> /GND
- U12 pad 4: Net-(J13-Pad2) -> /GND
- U13 pad 4: Net-(J14-Pad2) -> /GND
- U14 pad 4: Net-(J15-Pad2) -> /GND
- U15 pad 4: Net-(J16-Pad2) -> /GND
- U16 pad 4: Net-(J17-Pad2) -> /GND
- U17 pad 4: Net-(J18-Pad2) -> /GND
- U18 pad 4: Net-(J19-Pad2) -> /GND
- U19 pad 4: Net-(J20-Pad2) -> /GND
- U2 pad 4: Net-(J3-Pad2) -> /GND
- U20 pad 4: Net-(J21-Pad2) -> /GND
- U3 pad 4: Net-(J4-Pad2) -> /GND
- U4 pad 4: Net-(J5-Pad2) -> /GND
- U5 pad 4: Net-(J6-Pad2) -> /GND
- U6 pad 4: Net-(J7-Pad2) -> /GND
- U7 pad 4: Net-(J8-Pad2) -> /GND
- U8 pad 4: Net-(J9-Pad2) -> /GND
- U9 pad 4: Net-(J10-Pad2) -> /GND
Routing:
- net /5V: track 1333.9 -> 2.25 mm
- net /GND: track 1293.2 -> 22.8 mm
- net Net-(J5-Pad2): track 21.9 -> 0.00 mm
- net Net-(J20-Pad2): track 21.2 -> 0.00 mm
- net Net-(J2-Pad2): track 20.5 -> 0.00 mm
- net Net-(J4-Pad2): track 20.4 -> 0.00 mm
- net Net-(J17-Pad2): track 20.0 -> 0.00 mm
- net Net-(J19-Pad2): track 19.9 -> 0.00 mm
- net Net-(J18-Pad2): track 19.6 -> 0.00 mm
- net Net-(J12-Pad2): track 19.5 -> 0.00 mm
- net Net-(J13-Pad2): track 19.5 -> 0.00 mm
- net Net-(J15-Pad2): track 19.5 -> 0.00 mm
- net Net-(J11-Pad2): track 19.3 -> 0.00 mm
- net Net-(J8-Pad2): track 19.2 -> 0.00 mm
- net Net-(J14-Pad2): track 19.2 -> 0.00 mm
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- added copper zone on F.Cu, net /5V
- added copper zone on B.Cu, net /GND
Other:
- board text added: "IRIDIA"
- board text added: "e-puck extension battery charger V1.0"
